File: main_board/main_board.kicad_sch (KiCad schematic)
At the start: 68 parts, among them J1 3.5mm Jack, J18 Conn_01x15_Female, J19 Conn_01x15_Female, J2 3.5mm Jack, J3 3.5mm Jack, J4 3.5mm Jack, J5 Display Header, J6 EU Power, J7 Expansion Header, SW1 Push Button, SW10 Push Button, SW11 Push Button, SW12 Push Button, SW13 Push Button, SW14 Push Button, SW15 Push Button, SW16 Push Button, SW17 Push Button, SW2 Push Button, SW3 Push Button, SW4 Push Button, SW5 Adj, SW6 Push Button, SW7 Push Button, SW8 Push Button, SW9 Push Button, U14 MCP23008-xSO, U3 CD4013BPWR, U4 CD4013BPWR

Commit message: Ver 2.0 of board.
Also major advances in code.
Parts:
- removed C31: 100nF, Capacitor_SMD:C_0805_2012Metric_Pad1.18x1.45mm_HandSolder, symbol Device:C_Small
- removed U14: MCP23008-xSO, Package_SO:SOIC-18W_7.5x11.6mm_P1.27mm, symbol Interface_Expansion:MCP23008-xSO
- removed U3, U4: CD4013BPWR, Package_SO:TSSOP-14_4.4x5mm_P0.65mm, symbol 4xxx_IEEE:4013
- added C34: 100nF, Capacitor_SMD:C_0805_2012Metric_Pad1.18x1.45mm_HandSolder, symbol Device:C_Small
- added J20: Conn_01x02_Male, Connector_PinHeader_2.54mm:PinHeader_1x02_P2.54mm_Vertical, symbol Connector:Conn_01x02_Male
- added R125, R126, R127, R128, R56, R57, R58, R59, R60, R61, R66, R67, R68: 10K, Resistor_SMD:R_0805_2012Metric_Pad1.20x1.40mm_HandSolder, symbol Device:R_Small_US
- added R62, R63: 1M, Resistor_SMD:R_0805_2012Metric_Pad1.20x1.40mm_HandSolder, symbol Device:R_Small_US
- added R64, R65: 100K, Resistor_SMD:R_0805_2012Metric_Pad1.20x1.40mm_HandSolder, symbol Device:R_Small_US
- added U16: MB85RC256, Package_SO:SOIC-8_3.9x4.9mm_P1.27mm, symbol Memory_NVRAM:FM24C64B
- added U3: 74LVC07, Package_SO:TSSOP-14_4.4x5mm_P0.65mm, symbol 74xx:74LCX07
- A1: value Arduino_Nano_v3.x-MCU_Module -> Arduino_Nano_RP2040_Connect
Connections:
- net DIN is gone; now on net CS: A1.10 (D7), J18.10 (Pin_10)
- net KEYBINT is gone; now on net A: A1.8 (D5), J18.8 (Pin_8)
- net R0 is gone; now on net B0: A1.19 (A0), J19.12 (Pin_12)
- net R1 is gone; now on net B1: A1.20 (A1), J19.11 (Pin_11)
- net R2 is gone; now on net K0: A1.21 (A2), J19.10 (Pin_10)
- net R3 is gone; now on net K1: A1.22 (A3), J19.9 (Pin_9)
- net +3V3: now also C34.1, R125.1, R126.1, R127.1, R128.1, R56.2, R57.2, R58.2, R59.2, R60.1, R61.2, R66.1, R67.1, R68.1, U16.8 (VDD), U3.14 (VCC); no longer C30.1, SW1.1 (A), SW2.1 (A), SW3.1 (A), SW4.1 (A)
- net A: now also R60.2, R62.2, U3.10; no longer A1.5 (D2), C12.1, J18.5 (Pin_5), SW5.A
- net B: now also A1.9 (D6), J18.9 (Pin_9), R61.1, R63.2, U3.12; no longer A1.6 (D3), C11.1, J18.6 (Pin_6), SW5.B
- net CS: no longer A1.9 (D6), J18.9 (Pin_9)
- net GND: now also SW1.1 (A), SW2.1 (A), SW3.1 (A), SW4.1 (A), SW6.1 (A), SW7.1 (A), SW8.1 (A), SW9.1 (A), C34.2, J20.1 (Pin_1), U16.4 (VSS), U3.7 (GND)
- net P: now also C30.1, R68.2
- net Reset: no longer A1.28 (RESET), J19.3 (Pin_3)
- net SCL: now also U16.6 (SCL)
- net SDA: now also U16.5 (SDA)
- net T0: now also SW1.2 (B), R56.1, U3.2
- net T1: now also SW2.2 (B), R57.1, U3.4
- net T2: now also SW3.2 (B), R58.1, U3.6
- net T2 LED: now also A1.5 (D2), J18.6 (Pin_6); no longer A1.25 (A6), J19.6 (Pin_6)
- net T3: now also SW4.2 (B), R59.1, U3.8
- net T3 LED: now also A1.6 (D3), J18.5 (Pin_5); no longer A1.26 (A7), J19.5 (Pin_5)
- net at D4.1 (K), D8.2 (A), R4.1: now also U3.9; no longer SW4.2 (B)
- net B0: now reaches SW10.1 (A), SW11.1 (A), SW12.1 (A), SW13.1 (A)
- net B1: now reaches SW14.1 (A), SW15.1 (A), SW16.1 (A), SW17.1 (A)
- net K0: now reaches SW10.2 (B), SW14.2 (B), SW6.2 (B)
- net K0: now also R125.2
- net K1: now reaches SW11.2 (B), SW15.2 (B), SW7.2 (B)
- net K1: now also R126.2
- net K2: now reaches SW12.2 (B), SW16.2 (B), SW8.2 (B)
- net K2: now also A1.25 (A6), J19.6 (Pin_6), R127.2
- net K3: now reaches SW13.2 (B), SW17.2 (B), SW9.2 (B)
- net K3: now also A1.26 (A7), J19.5 (Pin_5), R128.2
- net at D2.1 (K), D7.2 (A), R2.1: now also U3.5; no longer SW3.2 (B)
- net at D3.1 (K), D6.2 (A), R3.1: now also U3.3; no longer SW2.2 (B)
- net at D1.1 (K), D5.2 (A), R1.1: now also U3.1; no longer SW1.2 (B)
- net 3.3VRef: no longer names the net of A1.18 (AREF)
- net 3.3VRef: no longer J19.13 (Pin_13)
- new net: C12.1, R65.1, R67.2, SW5.A
- new net: R63.1, R64.2, U3.13
- new net: R62.1, R65.2, U3.11
- new net: J19.3 (Pin_3), J20.2 (Pin_2)
- new net: C11.1, R64.1, R66.2, SW5.B
Other:
- added sheet Output Monitors (output_monitors.kicad_sch)
- note added: "Force Bootloader"
- moved on the sheet: A1, C11, C12, C7, D1, D10, D11, D12, D5, D9, J1, J18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

Commit message: Version 0.03
Parts:
- removed C23: 100nF, Capacitor_SMD:C_0805_2012Metric_Pad1.18x1.45mm_HandSolder, symbol Device:C_Small
- removed R56, R57, R58, R59, R60, R61: 10K, Resistor_SMD:R_0805_2012Metric_Pad1.20x1.40mm_HandSolder, symbol Device:R_Small_US
- removed R62, R63: 1M, Resistor_SMD:R_0805_2012Metric_Pad1.20x1.40mm_HandSolder, symbol Device:R_Small_US
- removed R64, R65: 100K, Resistor_SMD:R_0805_2012Metric_Pad1.20x1.40mm_HandSolder, symbol Device:R_Small_US
- removed U3: 74LVC07, Package_SO:TSSOP-14_4.4x5mm_P0.65mm, symbol 74xx:74LCX07
- added SO1, SO2, SO3, SO4: LED_Standoff, symbol greenface:LED_Standoff
- R5, R6, R7, R8: value 1K -> 300;  LCSC Part # C100047 -> C134081
Connections:
- net +3V3: now also SW1.2 (B), SW2.2 (B), SW3.2 (B), SW4.2 (B)
- net A: now also C12.1, R67.2, SW5.A
- net B: now also C11.1, R66.2, SW5.B
- net GND: no longer SW1.1 (A), SW2.1 (A), SW3.1 (A), SW4.1 (A)
- net T0: now also D1.1 (K), D5.2 (A), R1.1, SW1.1 (A); no longer SW1.2 (B)
- net T1: now also D3.1 (K), D6.2 (A), R3.1, SW2.1 (A); no longer SW2.2 (B)
- net T2: now also D2.1 (K), D7.2 (A), R2.1, SW3.1 (A); no longer SW3.2 (B)
- net T2 LED: now also J18.5 (Pin_5); no longer J18.6 (Pin_6)
- net T3: now also D4.1 (K), D8.2 (A), R4.1, SW4.1 (A); no longer SW4.2 (B)
- net T3 LED: now also J18.6 (Pin_6); no longer J18.5 (Pin_5)
Other:
- moved on the sheet: C11, C12, C30, D1, D2, D3, D4, D5, D6, D7, D8, R66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

Commit message: Version .20
Moves to external library
Parts:
- added N1, N2, N3, N4, N5, N6: Nut, symbol greenface:LED_Standoff
- added SC1, SC2, SC3, SC4: Screw, symbol greenface:LED_Standoff
- added SO25, SO26, SO27, SO28: Board Standoff, symbol greenface:LED_Standoff
- added SO29, SO30: DisplayStandoff, symbol greenface:LED_Standoff
- D10: Digi-Key Part 160-1035-ND -> 160-1961-ND
- D11: Digi-Key Part 160-1035-ND -> 732-5005-ND
- D12: Digi-Key Part 160-1035-ND -> 732-5008-ND
- D9: Digi-Key Part 160-1035-ND -> 732-11401-ND
Other:
- moved on the sheet: J7, SO1, SO2, SO3, SO4

Commit message: Software v2.2
Removes unneeded files.
Adds pre-flight handler in WiFi do_server();
Removes debug printouts.
Parts:
- J20:  LCSC Part # (none) -> C492401
Changed lines of the file:
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@@
+      (effects (font (size 1.27 1.27)) hide)
+    )
+    (property " LCSC Part #" "C492401" (id 5) (at 120.015 24.765 0)
       (effects (font (size 1.27 1.27)) hide)
     )
@@
     )
     (path "/eae55a42-d110-46e1-b06f-560b3d6a7f91/c48ee5e9-0cb9-42be-91f7-fd1b8daadc67"
-      (reference "R93") (unit 1) (value "56K") (footprint "Resistor_SMD:R_0805_2012Metric_Pad1.20x1.40mm_HandSolder")
+      (reference "R93") (unit 1) (value "100K") (footprint "Resistor_SMD:R_0805_2012Metric_Pad1.20x1.40mm_HandSolder")
     )
     (path "/eae55a42-d110-46e1-b06f-560b3d6a7f91/8f467469-5b59-49bc-9a45-5c4c02cfd83f"
-      (reference "R94") (unit 1) (value "56K") (footprint "Resistor_SMD:R_0805_2012Metric_Pad1.20x1.40mm_HandSolder")
+      (reference "R94") (unit 1) (value "100K") (footprint "Resistor_SMD:R_0805_2012Metric_Pad1.20x1.40mm_HandSolder")
     )
     (path "/eae55a42-d110-46e1-b06f-560b3d6a7f91/28bf7470-e1d2-4e98-a4b6-f98eb30a5a64"
-      (reference "R95") (unit 1) (value "56K") (footprint "Resistor_SMD:R_0805_2012Metric_Pad1.20x1.40mm_HandSolder")
+      (reference "R95") (unit 1) (value "100K") (footprint "Resistor_SMD:R_0805_2012Metric_Pad1.20x1.40mm_HandSolder")
     )
     (path "/eae55a42-d110-46e1-b06f-560b3d6a7f91/1e88784e-1b90-44c4-aa24-62abd646680b"
-      (reference "R96") (unit 1) (value "56K") (footprint "Resistor_SMD:R_0805_2012Metric_Pad1.20x1.40mm_HandSolder")
+      (reference "R96") (unit 1) (value "100K") (footprint "Resistor_SMD:R_0805_2012Metric_Pad1.20x1.40mm_HandSolder")
     )
     (path "/eae55a42-d110-46e1-b06f-560b3d6a7f91/af0f4f1e-590a-4e44-bb6f-03e1b7a33730"
@@
     )
     (path "/eae55a42-d110-46e1-b06f-560b3d6a7f91/5392f86f-026a-44a3-8a1d-a0c922c48ed1"
-      (reference "R121") (unit 1) (value "56K") (footprint "Resistor_SMD:R_0805_2012Metric_Pad1.20x1.40mm_HandSolder")
+      (reference "R121") (unit 1) (value "100K") (footprint "Resistor_SMD:R_0805_2012Metric_Pad1.20x1.40mm_HandSolder")
     )
     (path "/eae55a42-d110-46e1-b06f-560b3d6a7f91/d5a79db5-b8c5-4dbc-8d68-88add333d998"
-      (reference "R122") (unit 1) (value "56K") (footprint "Resistor_SMD:R_0805_2012Metric_Pad1.20x1.40mm_HandSolder")
+      (reference "R122") (unit 1) (value "100K") (footprint "Resistor_SMD:R_0805_2012Metric_Pad1.20x1.40mm_HandSolder")
     )
     (path "/eae55a42-d110-46e1-b06f-560b3d6a7f91/758ac2e7-692f-4be8-92b8-a60d9b85da79"
-      (reference "R123") (unit 1) (value "56K") (footprint "Resistor_SMD:R_0805_2012Metric_Pad1.20x1.40mm_HandSolder")
+      (reference "R123") (unit 1) (value "100K") (footprint "Resistor_SMD:R_0805_2012Metric_Pad1.20x1.40mm_HandSolder")
     )
     (path "/eae55a42-d110-46e1-b06f-560b3d6a7f91/3d08366c-664c-49aa-9264-fe38e52d7908"
-      (reference "R124") (unit 1) (value "56K") (footprint "Resistor_SMD:R_0805_2012Metric_Pad1.20x1.40mm_HandSolder")
+      (reference "R124") (unit 1) (value "100K") (footprint "Resistor_SMD:R_0805_2012Metric_Pad1.20x1.40mm_HandSolder")
     )
     (path "/b12871f3-737e-47b7-9f4c-ecb6eabe1783"
@@
     )
     (path "/808a57ff-0ced-4535-b028-9fea6b6c5f09/36580576-1e78-433f-b141-eb68f497b9e6"
-      (reference "R139") (unit 1) (value "56K") (footprint "Resistor_SMD:R_0805_2012Metric_Pad1.20x1.40mm_HandSolder")
+      (reference "R139") (unit 1) (value "100K") (footprint "Resistor_SMD:R_0805_2012Metric_Pad1.20x1.40mm_HandSolder")
     )
     (path "/808a57ff-0ced-4535-b028-9fea6b6c5f09/b8029def-cd05-4fce-a794-515779c7678d"
-      (reference "R140") (unit 1) (value "56K") (footprint "Resistor_SMD:R_0805_2012Metric_Pad1.20x1.40mm_HandSolder")
+      (reference "R140") (unit 1) (value "100K") (footprint "Resistor_SMD:R_0805_2012Metric_Pad1.20x1.40mm_HandSolder")
     )
     (path "/b200c1d4-b772-4a0d-a7bc-c10bcb241496/fce33d75-d8cb-456f-b73c-6382e195250c"

Commit message: Updates monitor circuitry. Sets outputs on init().
Parts:
- C1, C2:  LCSC Part # C2887276 -> C2887272
- C11, C12:  LCSC Part # C83170 -> C1710
- C7: value 330nF -> 1uF;  LCSC Part # C107132 -> C28323
- D1, D13, D14, D2, D3, D4, D5, D6, D7, D8: value BAT46 -> 1N5819;  LCSC Part # C123899 -> C191023
- R1, R125, R126, R127, R128, R2, R3, R4, R66, R67, R68:  LCSC Part # C138260 -> C17414
- R5, R6, R7, R8:  LCSC Part # C134081 -> C17617

Commit message: Upgrades board to v5. Adds Bonk Daddy.
Parts:
- added TP4: TestPoint, TestPoint:TestPoint_Keystone_5000-5004_Miniature, symbol Connector:TestPoint
- TP1, TP2:  LCSC Part # (none) -> C2906764
Connections:
- net CS: now also TP4.1
Other:
- title: (none) -> Bonkulator

Commit message: Adds 2HP BonkDaddy. Fixes boms/cpl. Updates Readme
Parts:
- added J21: OLED Pins, symbol dk_Rectangular-Connectors-Headers-Male-Pins:0022232041
- added M1: OLED, symbol greenface-symbols:OLED_Module
- J18, J19:  LCSC Part # C124408 -> C2932676
Changed lines of the file:
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@@
     (pin "2")
+  )
+  (symbol (lib_id "greenface-symbols:OLED_Module") (at 221.615 128.27 0) (unit 1)
+    (in_bom yes) (on_board no)
+    (property "Reference" "M1" (id 0) (at 228.6762 122.0216 0)
+      (effects (font (size 1.27 1.27)) (justify left))
+    )
+    (property "Value" "OLED" (id 1) (at 228.6762 124.333 0)
+      (effects (font (size 1.27 1.27)) (justify left))
+    )
+    (property "Footprint" "" (id 2) (at 221.615 128.27 0)
+      (effects (font (size 1.27 1.27)) hide)
+    )
+    (property "Datasheet" "" (id 3) (at 221.615 128.27 0)
+      (effects (font (size 1.27 1.27)) hide)
+    )
+    (property "URL" "https://www.amazon.com/gp/product/B072Q2X2LL/" (id 4) (at 221.615 128.27 0)
+      (effects (font (size 1.27 1.27)) hide)
+    )
   )
   (symbol (lib_id "greenface:LED_Standoff") (at 189.23 142.875 0) (unit 1)
@@
       (effects (font (size 1.27 1.27)) hide)
     )
-    (property " LCSC Part #" "C124408" (id 4) (at 95.25 48.26 0)
+    (property " LCSC Part #" "C2932676" (id 4) (at 95.25 48.26 0)
       (effects (font (size 1.27 1.27)) hide)
     )
@@
       (effects (font (size 1.27 1.27)) hide)
     )
-    (property " LCSC Part #" "C124408" (id 4) (at 99.695 48.26 0)
+    (property " LCSC Part #" "C2932676" (id 4) (at 99.695 48.26 0)
       (effects (font (size 1.27 1.27)) hide)
     )
@@
     (pin "2")
   )
+  (symbol (lib_id "dk_Rectangular-Connectors-Headers-Male-Pins:0022232041") (at 217.805 132.08 0) (mirror x) (unit 1)
+    (in_bom yes) (on_board no)
+    (property "Reference" "J21" (id 0) (at 231.775 130.175 0)
+      (effects (font (size 1.27 1.27)) (justify right))
+    )
+    (property "Value" "OLED Pins" (id 1) (at 238.125 132.08 0)
+      (effects (font (size 1.27 1.27)) (justify right))
+    )
+    (property "Footprint" "" (id 2) (at 222.885 137.16 0)
+      (effects (font (size 1.524 1.524)) (justify left) hide)
+    )
+    (property "Datasheet" "" (id 3) (at 222.885 139.7 0)
+      (effects (font (size 1.524 1.524)) (justify left) hide)
+    )
+    (property "Digi-Key Part" "732-5317-ND" (id 4) (at 222.885 142.24 0)
+      (effects (font (size 1.524 1.524)) (justify left) hide)
+    )
+    (pin "1")
+    (pin "2")
+    (pin "3")
+    (pin "4")
+  )
   (symbol (lib_id "power:+3.3V") (at 55.88 154.94 0) (unit 1)
     (in_bom yes) (on_board yes)
@@
     )
     (path "/b200c1d4-b772-4a0d-a7bc-c10bcb241496/0c7904aa-0aae-4e14-a46e-a653de8e9748"
-      (reference "#PWR?") (unit 1) (value "GND") (footprint "")
+      (reference "#PWR0121") (unit 1) (value "GND") (footprint "")
     )
     (path "/00000000-0000-0000-0000-0000623f6295"
@@
       (reference "J20") (unit 1) (value "Conn_01x02_Male") (footprint "Connector_PinHeader_2.54mm:PinHeader_1x02_P2.54mm_Vertical")
     )
+    (path "/9918d358-4286-4a0e-b531-5d4ecad91743"
+      (reference "J21") (unit 1) (value "OLED Pins") (footprint "")
+    )
+    (path "/21fca4dc-ad80-48a9-b01d-afbdf5accd55"
+      (reference "M1") (unit 1) (value "OLED") (footprint "")
+    )
     (path "/61c233db-1ac3-4100-988c-9d84873f2d10"
