File: main_board/outputs.kicad_sch (KiCad schematic)
At the start: 101 parts, among them J10 3.5mm Jack, J11 3.5mm Jack, J12 3.5mm Jack, J13 3.5mm Jack, J14 3.5mm Jack, J15 3.5mm Jack, J8 3.5mm Jack, J9 3.5mm Jack, Q1 MMBT3904, U1 TL072CDR, U13 DG412xY, U15 AS431, U2 TL072CDR, U21 MCP23008-xSS, U24 DG412xY, U5 TL072CDR, U6 AD5328, U8 TL072CDR, U9 TL072CDR

Commit message: Rev 4.2 of board
Parts:
- U13, U24: value DG412xY -> DG412DY-E3; LCSC Part # C143730 -> C45218
Changed lines of the file:
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@@
     (in_bom yes) (on_board yes)
     (property "Reference" "U24" (id 0) (at 192.405 74.295 0))
-    (property "Value" "DG412xY" (id 1) (at 191.77 76.835 0))
+    (property "Value" "DG412DY-E3" (id 1) (at 191.77 76.835 0))
     (property "Footprint" "Package_SO:SOIC-16_3.9x9.9mm_P1.27mm" (id 2) (at 198.755 74.93 0)
       (effects (font (size 1.27 1.27)) hide)
@@
       (effects (font (size 1.27 1.27)) hide)
     )
-    (property "LCSC Part #" "C143730" (id 4) (at 198.755 72.39 0)
+    (property "LCSC Part #" "C45218" (id 4) (at 198.755 72.39 0)
       (effects (font (size 1.27 1.27)) hide)
     )
@@
     (in_bom yes) (on_board yes)
     (property "Reference" "U24" (id 0) (at 192.405 120.65 0))
-    (property "Value" "DG412xY" (id 1) (at 191.77 123.19 0))
+    (property "Value" "DG412DY-E3" (id 1) (at 191.77 123.19 0))
     (property "Footprint" "Package_SO:SOIC-16_3.9x9.9mm_P1.27mm" (id 2) (at 198.755 121.285 0)
       (effects (font (size 1.27 1.27)) hide)
@@
       (effects (font (size 1.27 1.27)) hide)
     )
-    (property "LCSC Part #" "C143730" (id 4) (at 198.755 118.745 0)
+    (property "LCSC Part #" "C45218" (id 4) (at 198.755 118.745 0)
       (effects (font (size 1.27 1.27)) hide)
     )
@@
     (in_bom yes) (on_board yes)
     (property "Reference" "U13" (id 0) (at 20.955 133.985 0))
-    (property "Value" "DG412xY" (id 1) (at 19.685 137.16 0))
+    (property "Value" "DG412DY-E3" (id 1) (at 19.685 137.16 0))
     (property "Footprint" "Package_SO:SOIC-16_3.9x9.9mm_P1.27mm" (id 2) (at 30.48 140.335 0)
       (effects (font (size 1.27 1.27)) hide)
@@
       (effects (font (size 1.27 1.27)) hide)
     )
-    (property "LCSC Part #" "C143730" (id 4) (at 30.48 137.795 0)
+    (property "LCSC Part #" "C45218" (id 4) (at 30.48 137.795 0)
       (effects (font (size 1.27 1.27)) hide)
     )
@@
     (in_bom yes) (on_board yes)
     (property "Reference" "U13" (id 0) (at 84.455 121.92 0))
-    (property "Value" "DG412xY" (id 1) (at 83.82 124.46 0))
+    (property "Value" "DG412DY-E3" (id 1) (at 83.82 124.46 0))
     (property "Footprint" "Package_SO:SOIC-16_3.9x9.9mm_P1.27mm" (id 2) (at 90.805 122.555 0)
       (effects (font (size 1.27 1.27)) hide)
@@
       (effects (font (size 1.27 1.27)) hide)
     )
-    (property "LCSC Part #" "C143730" (id 4) (at 90.805 120.015 0)
+    (property "LCSC Part #" "C45218" (id 4) (at 90.805 120.015 0)
       (effects (font (size 1.27 1.27)) hide)
     )
@@
     (in_bom yes) (on_board yes)
     (property "Reference" "U13" (id 0) (at 84.455 97.79 0))
-    (property "Value" "DG412xY" (id 1) (at 83.82 100.33 0))
+    (property "Value" "DG412DY-E3" (id 1) (at 83.82 100.33 0))
     (property "Footprint" "Package_SO:SOIC-16_3.9x9.9mm_P1.27mm" (id 2) (at 90.805 98.425 0)
       (effects (font (size 1.27 1.27)) hide)
@@
       (effects (font (size 1.27 1.27)) hide)
     )
-    (property "LCSC Part #" "C143730" (id 4) (at 90.805 95.885 0)
+    (property "LCSC Part #" "C45218" (id 4) (at 90.805 95.885 0)
       (effects (font (size 1.27 1.27)) hide)
     )
@@
     (in_bom yes) (on_board yes)
     (property "Reference" "U24" (id 0) (at 20.32 170.18 0))
-    (property "Value" "DG412xY" (id 1) (at 19.05 173.355 0))
+    (property "Value" "DG412DY-E3" (id 1) (at 19.05 173.355 0))
     (property "Footprint" "Package_SO:SOIC-16_3.9x9.9mm_P1.27mm" (id 2) (at 29.845 176.53 0)
       (effects (font (size 1.27 1.27)) hide)
@@
       (effects (font (size 1.27 1.27)) hide)
     )
-    (property "LCSC Part #" "C143730" (id 4) (at 29.845 173.99 0)
+    (property "LCSC Part #" "C45218" (id 4) (at 29.845 173.99 0)
       (effects (font (size 1.27 1.27)) hide)
     )
@@
     (in_bom yes) (on_board yes)
     (property "Reference" "U13" (id 0) (at 84.455 146.05 0))
-    (property "Value" "DG412xY" (id 1) (at 83.82 148.59 0))
+    (property "Value" "DG412DY-E3" (id 1) (at 83.82 148.59 0))
     (property "Footprint" "Package_SO:SOIC-16_3.9x9.9mm_P1.27mm" (id 2) (at 90.805 146.685 0)
       (effects (font (size 1.27 1.27)) hide)
@@
       (effects (font (size 1.27 1.27)) hide)
     )
-    (property "LCSC Part #" "C143730" (id 4) (at 90.805 144.145 0)
+    (property "LCSC Part #" "C45218" (id 4) (at 90.805 144.145 0)
       (effects (font (size 1.27 1.27)) hide)
     )
@@
     (in_bom yes) (on_board yes)
     (property "Reference" "U24" (id 0) (at 192.405 96.52 0))
-    (property "Value" "DG412xY" (id 1) (at 191.77 99.06 0))
+    (property "Value" "DG412DY-E3" (id 1) (at 191.77 99.06 0))
     (property "Footprint" "Package_SO:SOIC-16_3.9x9.9mm_P1.27mm" (id 2) (at 198.755 97.155 0)
       (effects (font (size 1.27 1.27)) hide)
@@
       (effects (font (size 1.27 1.27)) hide)
     )
-    (property "LCSC Part #" "C143730" (id 4) (at 198.755 94.615 0)
+    (property "LCSC Part #" "C45218" (id 4) (at 198.755 94.615 0)
       (effects (font (size 1.27 1.27)) hide)
     )
@@
     (in_bom yes) (on_board yes)
     (property "Reference" "U13" (id 0) (at 84.455 76.2 0))
-    (property "Value" "DG412xY" (id 1) (at 83.82 78.74 0))
+    (property "Value" "DG412DY-E3" (id 1) (at 83.82 78.74 0))
     (property "Footprint" "Package_SO:SOIC-16_3.9x9.9mm_P1.27mm" (id 2) (at 90.805 76.835 0)
       (effects (font (size 1.27 1.27)) hide)
@@
       (effects (font (size 1.27 1.27)) hide)
     )
-    (property "LCSC Part #" "C143730" (id 4) (at 90.805 74.295 0)
+    (property "LCSC Part #" "C45218" (id 4) (at 90.805 74.295 0)
       (effects (font (size 1.27 1.27)) hide)
     )
@@
     (in_bom yes) (on_board yes)
     (property "Reference" "U24" (id 0) (at 192.405 144.78 0))
-    (property "Value" "DG412xY" (id 1) (at 191.77 147.32 0))
+    (property "Value" "DG412DY-E3" (id 1) (at 191.77 147.32 0))
     (property "Footprint" "Package_SO:SOIC-16_3.9x9.9mm_P1.27mm" (id 2) (at 198.755 145.415 0)
       (effects (font (size 1.27 1.27)) hide)
@@
       (effects (font (size 1.27 1.27)) hide)
     )
-    (property "LCSC Part #" "C143730" (id 4) (at 198.755 142.875 0)
-      (effects (font (size 1.27 1.27)) hide)
-    )
+    (property "LCSC Part #" "C45218" (id 4) (at 198.755 142.875 0)
+      (effects (font (size 1.27 1.27)) hide)
+    )
