File: main_board/outputs.kicad_sch (KiCad schematic)
At the start: 101 parts, among them J10 3.5mm Jack, J11 3.5mm Jack, J12 3.5mm Jack, J13 3.5mm Jack, J14 3.5mm Jack, J15 3.5mm Jack, J8 3.5mm Jack, J9 3.5mm Jack, Q1 MMBT3904, U1 TL072CDR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

Commit message: Updates board to 5.0
Adds output resistors. Fixes AS431 pinout
Parts:
- removed U15: AS431, Package_TO_SOT_SMD:SOT-23, symbol Reference_Voltage:TL431DBZ
- added R81, R82, R83, R84, R85, R86, R87, R88: 1K, Resistor_SMD:R_0603_1608Metric, symbol Device:R_Small_US
- added U15: AS431HANTR, Package_TO_SOT_SMD:SOT-23, symbol greenface-symbols:AS431HANTR
- R76: LCSC Part # C21190 -> C2653986
- RV9: footprint sputterizer:Potentiometer_Bourns_3224W_Vertical -> Potentiometer_SMD:Potentiometer_Bourns_3224W_Vertical; LCSC Part # C780220 -> C81348
Connections:
- net 3.3VRef: now also U15.2 (K)
- net GND: now also U15.3 (A)
- net Out0: now also R81.2; no longer J8.2 (T)
- net Out1: now also R84.2; no longer J9.2 (T)
- net Out2: now also R82.2; no longer J10.2 (T)
- net Out3: now also R83.2; no longer J11.2 (T)
- net Out4: now also R87.2; no longer J12.2 (T)
- net Out5: now also R85.2; no longer J13.2 (T)
- net Out6: now also R86.2; no longer J14.2 (T)
- net Out7: now also R88.2; no longer J15.2 (T)
- net at R77.1, R78.1: now also U15.1 (REF)
- new net: J15.2 (T), R88.1
- new net: J13.2 (T), R85.1
- new net: J9.2 (T), R84.1
- new net: J10.2 (T), R82.1
- new net: J8.2 (T), R81.1
- new net: J11.2 (T), R83.1
- new net: J12.2 (T), R87.1
- new net: J14.2 (T), R86.1
Other:
- note added: "3224w"
- note removed: "3314G"
- moved on the sheet: RV9

Commit message: Either Way doesn't work
Saved just in case
Parts:
- removed R81, R82, R83, R84, R85, R86, R87, R88: 1K, Resistor_SMD:R_0603_1608Metric, symbol Device:R_Small_US
Connections:
- net Out0: now also J8.2 (T)
- net Out1: now also J9.2 (T)
- net Out2: now also J10.2 (T)
- net Out3: now also J11.2 (T)
- net Out4: now also J12.2 (T)
- net Out5: now also J13.2 (T)
- net Out6: now also J14.2 (T)
- net Out7: now also J15.2 (T)

Commit message: New layout. Fixes regulator chip pinout error.
Parts:
- C31: value 330nF -> 1uF; LCSC Part # C1740 -> C28323
- R141: value 20K -> 10K; Digi-Key Part RMCF0805JT20K0CT-ND -> 13-RC0805JR-1010KLCT-ND; LCSC Part # C4328 -> C17414
Changed lines of the file:
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@@
 (kicad_sch (version 20211123) (generator eeschema)
   (paper "A4")
+  (title_block
+    (rev "4.3")
+  )
   (junction (at 116.84 114.935) (diameter 0) (color 0 0 0 0)
   )
@@
       (effects (font (size 1.27 1.27)) (justify left))
     )
-    (property "Value" "330nF" (id 1) (at 128.27 45.085 0)
+    (property "Value" "1uF" (id 1) (at 125.73 44.45 0)
       (effects (font (size 1.27 1.27)) (justify left))
     )
@@
       (effects (font (size 1.27 1.27)) hide)
     )
-    (property "LCSC Part #" "C1740" (id 5) (at 119.38 42.545 0)
+    (property "LCSC Part #" "C28323" (id 5) (at 119.38 42.545 0)
       (effects (font (size 1.27 1.27)) hide)
     )
@@
     (in_bom yes) (on_board yes)
     (property "Reference" "R141" (id 0) (at 107.95 36.195 90))
-    (property "Value" "20K" (id 1) (at 107.95 41.275 90))
+    (property "Value" "10K" (id 1) (at 107.95 41.275 90))
     (property "Footprint" "Resistor_SMD:R_0805_2012Metric_Pad1.20x1.40mm_HandSolder" (id 2) (at 107.95 38.735 0)
       (effects (font (size 1.27 1.27)) hide)
@@
       (effects (font (size 1.27 1.27)) hide)
     )
-    (property "Digi-Key Part" "RMCF0805JT20K0CT-ND" (id 4) (at 107.95 38.735 90)
+    (property "Digi-Key Part" "13-RC0805JR-1010KLCT-ND" (id 4) (at 107.95 38.735 90)
       (effects (font (size 1.27 1.27)) hide)
     )
-    (property "LCSC Part #" "C4328" (id 5) (at 107.95 38.735 90)
+    (property "LCSC Part #" "C17414" (id 5) (at 107.95 38.735 90)
       (effects (font (size 1.27 1.27)) hide)
     )

Commit message: Fixes main board.
Fixes regulator footprint. Re lays out board to improve noise performance. Around -50db now at outputs.
Parts:
- Q1: LCSC Part # C94514 -> C20526
- R20, R21, R22, R23, R48, R49, R50, R51, R58: value 43K -> 33K; Digi-Key Part 311-43KARCT-ND -> RMCF0805JT33K0CT-ND; LCSC Part # C17695 -> C17633
- R24, R25, R26, R27, R52, R53, R54, R55: LCSC Part # C228750 -> C2681637
- R76: Digi-Key Part (none) -> RNCP0603FTD1K00CT-ND; LCSC Part # C2653986 -> C21190
- U15: Digi-Key Part (none) -> AS431HANTR-G1DICT-ND; LCSC Part # (none) -> C460669

Commit message: Updates bom for digi-key
Parts:
- C31, C43: Digi-Key Part 311-1888-1-ND -> 1276-1029-1-ND
- D43, D44: Digi-Key Part (none) -> DDZ7V5CDICT-ND
- Q1: Digi-Key Part (none) -> 4878-MMBT3904CT-ND
- R59, R60: Digi-Key Part RMCF0805JT20K0CT-ND -> 311-680ARCT-ND
- R77: Digi-Key Part (none) -> RMCF0603FT23K7CT-ND
- RV9: Digi-Key Part (none) -> 3224W-1-103GCT-ND
- U1, U2, U5, U8, U9: Digi-Key Part 296-47385-1-ND -> 296-1282-1-ND
- U13, U24: Digi-Key Part (none) -> DG412DY-E3-ND
Changed lines of the file:
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@@
+      (effects (font (size 1.27 1.27)) hide)
+    )
+    (property "Digi-Key Part" "DG412DY-E3-ND" (id 5) (at 198.755 72.39 0)
       (effects (font (size 1.27 1.27)) hide)
     )
@@
       (effects (font (size 1.27 1.27)) hide)
     )
-    (property "Digi-Key Part" "296-47385-1-ND" (id 4) (at 247.015 31.75 0)
+    (property "Digi-Key Part" "296-1282-1-ND" (id 4) (at 247.015 31.75 0)
       (effects (font (size 1.27 1.27)) hide)
     )
@@
       (effects (font (size 1.27 1.27)) hide)
     )
+    (property "Digi-Key Part" "DG412DY-E3-ND" (id 5) (at 198.755 118.745 0)
+      (effects (font (size 1.27 1.27)) hide)
+    )
     (pin "10")
     (pin "11")
@@
       (effects (font (size 1.27 1.27)) hide)
     )
-    (property "Digi-Key Part" "296-47385-1-ND" (id 4) (at 125.73 95.25 0)
+    (property "Digi-Key Part" "296-1282-1-ND" (id 4) (at 125.73 95.25 0)
       (effects (font (size 1.27 1.27)) hide)
     )
@@
       (effects (font (size 1.27 1.27)) hide)
     )
+    (property "Digi-Key Part" "DG412DY-E3-ND" (id 5) (at 30.48 137.795 0)
+      (effects (font (size 1.27 1.27)) hide)
+    )
     (pin "12")
     (pin "13")
@@
       (effects (font (size 1.27 1.27)) hide)
     )
+    (property "Digi-Key Part" "DDZ7V5CDICT-ND" (id 5) (at 63.5 166.37 0)
+      (effects (font (size 1.27 1.27)) hide)
+    )
     (pin "1")
     (pin "2")
@@
       (effects (font (size 1.27 1.27)) hide)
     )
-    (property "Digi-Key Part" "" (id 4) (at 157.48 32.385 90)
+    (property "Digi-Key Part" "RMCF0603FT23K7CT-ND" (id 4) (at 157.48 32.385 90)
       (effects (font (size 1.27 1.27)) hide)
     )
@@
       (effects (font (size 1.27 1.27)) hide)
     )
-    (property "Digi-Key Part" "296-47385-1-ND" (id 4) (at 95.25 173.355 0)
+    (property "Digi-Key Part" "296-1282-1-ND" (id 4) (at 95.25 173.355 0)
       (effects (font (size 1.27 1.27)) hide)
     )
@@
       (effects (font (size 1.27 1.27)) hide)
     )
-    (property "Digi-Key Part" "296-47385-1-ND" (id 4) (at 71.755 173.355 0)
+    (property "Digi-Key Part" "296-1282-1-ND" (id 4) (at 71.755 173.355 0)
       (effects (font (size 1.27 1.27)) hide)
     )
@@
       (effects (font (size 1.27 1.27)) hide)
     )
+    (property "Digi-Key Part" "DG412DY-E3-ND" (id 5) (at 90.805 120.015 0)
+      (effects (font (size 1.27 1.27)) hide)
+    )
     (pin "10")
     (pin "11")
@@
       (effects (font (size 1.27 1.27)) hide)
     )
+    (property "Digi-Key Part" "DG412DY-E3-ND" (id 5) (at 90.805 95.885 0)
+      (effects (font (size 1.27 1.27)) hide)
+    )
     (pin "6")
     (pin "7")
@@
     )
     (property "LCSC Part #" "C45218" (id 4) (at 29.845 173.99 0)
+      (effects (font (size 1.27 1.27)) hide)
+    )
+    (property "Digi-Key Part" "DG412DY-E3-ND" (id 5) (at 29.845 173.99 0)
       (effects (font (size 1.27 1.27)) hide)
     )
@@
       (effects (font (size 1.27 1.27)) hide)
     )
-    (property "Digi-Key Part" "296-47385-1-ND" (id 4) (at 207.645 36.83 0)
+    (property "Digi-Key Part" "296-1282-1-ND" (id 4) (at 207.645 36.83 0)
       (effects (font (size 1.27 1.27)) hide)
     )
@@
       (effects (font (size 1.27 1.27)) hide)
     )
+    (property "Digi-Key Part" "4878-MMBT3904CT-ND" (id 5) (at 119.38 31.75 0)
+      (effects (font (size 1.27 1.27)) hide)
+    )
     (pin "1")
     (pin "2")
@@
       (effects (font (size 1.27 1.27)) hide)
     )
-    (property "Digi-Key Part" "296-47385-1-ND" (id 4) (at 233.68 95.25 0)
+    (property "Digi-Key Part" "296-1282-1-ND" (id 4) (at 233.68 95.25 0)
       (effects (font (size 1.27 1.27)) hide)
     )
@@
       (effects (font (size 1.27 1.27)) hide)
     )
-    (property "Digi-Key Part" "296-47385-1-ND" (id 4) (at 125.73 119.38 0)
+    (property "Digi-Key Part" "296-1282-1-ND" (id 4) (at 125.73 119.38 0)
       (effects (font (size 1.27 1.27)) hide)
     )
@@
       (effects (font (size 1.27 1.27)) hide)
     )
-    (property "Digi-Key Part" "311-1888-1-ND" (id 4) (at 134.62 38.1 0)
+    (property "Digi-Key Part" "1276-1029-1-ND" (id 4) (at 134.62 38.1 0)
       (effects (font (size 1.27 1.27)) hide)
     )
@@
       (effects (font (size 1.27 1.27)) hide)
     )
-    (property "Digi-Key Part" "296-47385-1-ND" (id 4) (at 88.9 173.355 0)
+    (property "Digi-Key Part" "296-1282-1-ND" (id 4) (at 88.9 173.355 0)
       (effects (font (size 1.27 1.27)) hide)
     )
@@
       (effects (font (size 1.27 1.27)) hide)
     )
-    (property "Digi-Key Part" "296-47385-1-ND" (id 4) (at 125.73 143.51 0)
+    (property "Digi-Key Part" "296-1282-1-ND" (id 4) (at 125.73 143.51 0)
       (effects (font (size 1.27 1.27)) hide)
     )
@@
       (effects (font (size 1.27 1.27)) hide)
     )
+    (property "Digi-Key Part" "DG412DY-E3-ND" (id 5) (at 90.805 144.145 0)
+      (effects (font (size 1.27 1.27)) hide)
+    )
     (pin "14")
     (pin "15")
@@
       (effects (font (size 1.27 1.27)) hide)
     )
-    (property "Digi-Key Part" "RMCF0805JT20K0CT-ND" (id 4) (at 69.215 185.42 90)
+    (property "Digi-Key Part" "311-680ARCT-ND" (id 4) (at 69.215 185.42 90)
       (effects (font (size 1.27 1.27)) hide)
     )
@@
       (effects (font (size 1.27 1.27)) hide)
     )
-    (property "Digi-Key Part" "296-47385-1-ND" (id 4) (at 233.68 73.66 0)
+    (property "Digi-Key Part" "296-1282-1-ND" (id 4) (at 233.68 73.66 0)
       (effects (font (size 1.27 1.27)) hide)
     )
@@
       (effects (font (size 1.27 1.27)) hide)
     )
+    (property "Digi-Key Part" "DG412DY-E3-ND" (id 5) (at 198.755 94.615 0)
+      (effects (font (size 1.27 1.27)) hide)
+    )
     (pin "6")
     (pin "7")
@@
       (effects (font (size 1.27 1.27)) hide)
     )
-    (property "Digi-Key Part" "296-47385-1-ND" (id 4) (at 233.68 143.51 0)
+    (property "Digi-Key Part" "296-1282-1-ND" (id 4) (at 233.68 143.51 0)
       (effects (font (size 1.27 1.27)) hide)
     )
@@
       (effects (font (size 1.27 1.27)) hide)
     )
+    (property "Digi-Key Part" "3224W-1-103GCT-ND" (id 5) (at 157.48 22.86 0)
+      (effects (font (size 1.27 1.27)) hide)
+    )
     (pin "1")
     (pin "2")
@@
       (effects (font (size 1.27 1.27)) hide)
     )
-    (property "Digi-Key Part" "RMCF0805JT20K0CT-ND" (id 4) (at 69.215 161.29 90)
+    (property "Digi-Key Part" "311-680ARCT-ND" (id 4) (at 69.215 161.29 90)
       (effects (font (size 1.27 1.27)) hide)
     )
@@
       (effects (font (size 1.27 1.27)) hide)
     )
-    (property "Digi-Key Part" "296-47385-1-ND" (id 4) (at 233.68 119.38 0)
+    (property "Digi-Key Part" "296-1282-1-ND" (id 4) (at 233.68 119.38 0)
       (effects (font (size 1.27 1.27)) hide)
     )
@@
       (effects (font (size 1.27 1.27)) hide)
     )
-    (property "Digi-Key Part" "311-1888-1-ND" (id 4) (at 119.38 42.545 0)
+    (property "Digi-Key Part" "1276-1029-1-ND" (id 4) (at 119.38 42.545 0)
       (effects (font (size 1.27 1.27)) hide)
     )
@@
     )
     (property "LCSC Part #" "C545306" (id 4) (at 63.5 181.61 0)
+      (effects (font (size 1.27 1.27)) hide)
+    )
+    (property "Digi-Key Part" "DDZ7V5CDICT-ND" (id 5) (at 63.5 181.61 0)
       (effects (font (size 1.27 1.27)) hide)
     )
@@
       (effects (font (size 1.27 1.27)) hide)
     )
+    (property "Digi-Key Part" "DG412DY-E3-ND" (id 5) (at 90.805 74.295 0)
+      (effects (font (size 1.27 1.27)) hide)
+    )
     (pin "1")
     (pin "2")
@@
       (effects (font (size 1.27 1.27)) hide)
     )
-    (property "Digi-Key Part" "296-47385-1-ND" (id 4) (at 93.98 173.355 0)
+    (property "Digi-Key Part" "296-1282-1-ND" (id 4) (at 93.98 173.355 0)
       (effects (font (size 1.27 1.27)) hide)
     )
@@
       (effects (font (size 1.27 1.27)) hide)
     )
+    (property "Digi-Key Part" "DG412DY-E3-ND" (id 5) (at 198.755 142.875 0)
+      (effects (font (size 1.27 1.27)) hide)
+    )
     (pin "14")
     (pin "15")
@@
       (effects (font (size 1.27 1.27)) hide)
     )
-    (property "Digi-Key Part" "296-47385-1-ND" (id 4) (at 83.185 173.355 0)
+    (property "Digi-Key Part" "296-1282-1-ND" (id 4) (at 83.185 173.355 0)
       (effects (font (size 1.27 1.27)) hide)
     )
@@
       (effects (font (size 1.27 1.27)) hide)
     )
-    (property "Digi-Key Part" "296-47385-1-ND" (id 4) (at 125.73 73.66 0)
-      (effects (font (size 1.27 1.27)) hide)
-    )
+    (property "Digi-Key Part" "296-1282-1-ND" (id 4) (at 125.73 73.66 0)
+      (effects (font (size 1.27 1.27)) hide)
+    )
