File: main_board/triggers.kicad_sch (KiCad schematic)
At the start: 28 parts, among them J1 3.5mm Jack, J2 3.5mm Jack, J3 3.5mm Jack, J4 3.5mm Jack, SW1 Push Button, SW2 Push Button, SW3 Push Button, SW4 Push Button

Commit message: Fixes main board.
Fixes regulator footprint. Re lays out board to improve noise performance. Around -50db now at outputs.
Parts:
- R79, R80, R81, R82: Digi-Key Part (none) -> RNCP0603FTD1K00CT-ND; LCSC Part # C2653986 -> C21190
Changed lines of the file:
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@@
       (effects (font (size 1.27 1.27)) hide)
     )
-    (property "Digi-Key Part" "" (id 4) (at 74.93 54.61 90)
-      (effects (font (size 1.27 1.27)) hide)
-    )
-    (property "LCSC Part #" "C2653986" (id 5) (at 74.93 54.61 0)
+    (property "Digi-Key Part" "RNCP0603FTD1K00CT-ND" (id 4) (at 74.93 54.61 90)
+      (effects (font (size 1.27 1.27)) hide)
+    )
+    (property "LCSC Part #" "C21190" (id 5) (at 74.93 54.61 0)
       (effects (font (size 1.27 1.27)) hide)
     )
@@
       (effects (font (size 1.27 1.27)) hide)
     )
-    (property "Digi-Key Part" "" (id 4) (at 144.78 102.235 90)
-      (effects (font (size 1.27 1.27)) hide)
-    )
-    (property "LCSC Part #" "C2653986" (id 5) (at 144.78 102.235 0)
+    (property "Digi-Key Part" "RNCP0603FTD1K00CT-ND" (id 4) (at 144.78 102.235 90)
+      (effects (font (size 1.27 1.27)) hide)
+    )
+    (property "LCSC Part #" "C21190" (id 5) (at 144.78 102.235 0)
       (effects (font (size 1.27 1.27)) hide)
     )
@@
       (effects (font (size 1.27 1.27)) hide)
     )
-    (property "Digi-Key Part" "" (id 4) (at 144.78 55.245 90)
-      (effects (font (size 1.27 1.27)) hide)
-    )
-    (property "LCSC Part #" "C2653986" (id 5) (at 144.78 55.245 0)
+    (property "Digi-Key Part" "RNCP0603FTD1K00CT-ND" (id 4) (at 144.78 55.245 90)
+      (effects (font (size 1.27 1.27)) hide)
+    )
+    (property "LCSC Part #" "C21190" (id 5) (at 144.78 55.245 0)
       (effects (font (size 1.27 1.27)) hide)
     )
@@
       (effects (font (size 1.27 1.27)) hide)
     )
-    (property "Digi-Key Part" "" (id 4) (at 74.93 102.87 90)
-      (effects (font (size 1.27 1.27)) hide)
-    )
-    (property "LCSC Part #" "C2653986" (id 5) (at 74.93 102.87 0)
-      (effects (font (size 1.27 1.27)) hide)
-    )
+    (property "Digi-Key Part" "RNCP0603FTD1K00CT-ND" (id 4) (at 74.93 102.87 90)
+      (effects (font (size 1.27 1.27)) hide)
+    )
+    (property "LCSC Part #" "C21190" (id 5) (at 74.93 102.87 0)
+      (effects (font (size 1.27 1.27)) hide)
+    )
