File: main_board/inputs.kicad_sch (KiCad schematic)
At the start: 45 parts, among them J16 3.5mm Jack, J17 3.5mm Jack, U10 TL072CDR, U11 ADS1015IDGS, U12 TL072CDR, U19 TL072CDR

Commit message: Fixes main board.
Fixes regulator footprint. Re lays out board to improve noise performance. Around -50db now at outputs.
Parts:
- R30, R35: value 4.3K -> 4.7K; Digi-Key Part 311-43KARCT-ND -> RMCF0805FT4K70CT-ND; LCSC Part # C17667 -> C17673
- R38, R39: value 2.2K -> 10K; Digi-Key Part 311-10KARCT-ND -> 13-RC0805JR-1010KLCT-ND; LCSC Part # C17520 -> C17414
Changed lines of the file:
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@@
     (in_bom yes) (on_board yes)
     (property "Reference" "R38" (id 0) (at 100.33 71.12 90))
-    (property "Value" "2.2K" (id 1) (at 101.6 76.2 90))
+    (property "Value" "10K" (id 1) (at 101.6 76.2 90))
     (property "Footprint" "Resistor_SMD:R_0805_2012Metric_Pad1.20x1.40mm_HandSolder" (id 2) (at 100.33 73.66 0)
       (effects (font (size 1.27 1.27)) hide)
@@
       (effects (font (size 1.27 1.27)) hide)
     )
-    (property "Digi-Key Part" "311-10KARCT-ND" (id 4) (at 100.33 73.66 90)
-      (effects (font (size 1.27 1.27)) hide)
-    )
-    (property "LCSC Part #" "C17520" (id 5) (at 100.33 73.66 0)
+    (property "Digi-Key Part" "13-RC0805JR-1010KLCT-ND" (id 4) (at 100.33 73.66 90)
+      (effects (font (size 1.27 1.27)) hide)
+    )
+    (property "LCSC Part #" "C17414" (id 5) (at 100.33 73.66 0)
       (effects (font (size 1.27 1.27)) hide)
     )
@@
     (in_bom yes) (on_board yes)
     (property "Reference" "R30" (id 0) (at 104.775 53.34 90))
-    (property "Value" "4.3K" (id 1) (at 104.775 55.88 90))
+    (property "Value" "4.7K" (id 1) (at 104.775 55.88 90))
     (property "Footprint" "Resistor_SMD:R_0805_2012Metric_Pad1.20x1.40mm_HandSolder" (id 2) (at 104.775 50.8 0)
       (effects (font (size 1.27 1.27)) hide)
@@
       (effects (font (size 1.27 1.27)) hide)
     )
-    (property "Digi-Key Part" "311-43KARCT-ND" (id 4) (at 104.775 50.8 90)
-      (effects (font (size 1.27 1.27)) hide)
-    )
-    (property "LCSC Part #" "C17667" (id 5) (at 104.775 50.8 0)
+    (property "Digi-Key Part" "RMCF0805FT4K70CT-ND" (id 4) (at 104.775 50.8 90)
+      (effects (font (size 1.27 1.27)) hide)
+    )
+    (property "LCSC Part #" "C17673" (id 5) (at 104.775 50.8 0)
       (effects (font (size 1.27 1.27)) hide)
     )
@@
     (in_bom yes) (on_board yes)
     (property "Reference" "R39" (id 0) (at 101.6 140.335 90))
-    (property "Value" "2.2K" (id 1) (at 102.87 145.415 90))
+    (property "Value" "10K" (id 1) (at 102.87 145.415 90))
     (property "Footprint" "Resistor_SMD:R_0805_2012Metric_Pad1.20x1.40mm_HandSolder" (id 2) (at 101.6 142.875 0)
       (effects (font (size 1.27 1.27)) hide)
@@
       (effects (font (size 1.27 1.27)) hide)
     )
-    (property "Digi-Key Part" "311-10KARCT-ND" (id 4) (at 101.6 142.875 90)
-      (effects (font (size 1.27 1.27)) hide)
-    )
-    (property "LCSC Part #" "C17520" (id 5) (at 101.6 142.875 0)
+    (property "Digi-Key Part" "13-RC0805JR-1010KLCT-ND" (id 4) (at 101.6 142.875 90)
+      (effects (font (size 1.27 1.27)) hide)
+    )
+    (property "LCSC Part #" "C17414" (id 5) (at 101.6 142.875 0)
       (effects (font (size 1.27 1.27)) hide)
     )
@@
     (in_bom yes) (on_board yes)
     (property "Reference" "R35" (id 0) (at 104.775 122.555 90))
-    (property "Value" "4.3K" (id 1) (at 104.775 125.095 90))
+    (property "Value" "4.7K" (id 1) (at 104.775 125.095 90))
     (property "Footprint" "Resistor_SMD:R_0805_2012Metric_Pad1.20x1.40mm_HandSolder" (id 2) (at 104.775 120.015 0)
       (effects (font (size 1.27 1.27)) hide)
@@
       (effects (font (size 1.27 1.27)) hide)
     )
-    (property "Digi-Key Part" "311-43KARCT-ND" (id 4) (at 104.775 120.015 90)
-      (effects (font (size 1.27 1.27)) hide)
-    )
-    (property "LCSC Part #" "C17667" (id 5) (at 104.775 120.015 0)
-      (effects (font (size 1.27 1.27)) hide)
-    )
+    (property "Digi-Key Part" "RMCF0805FT4K70CT-ND" (id 4) (at 104.775 120.015 90)
+      (effects (font (size 1.27 1.27)) hide)
+    )
+    (property "LCSC Part #" "C17673" (id 5) (at 104.775 120.015 0)
+      (effects (font (size 1.27 1.27)) hide)
+    )

Commit message: Updates bom for digi-key
Parts:
- R28, R33: Digi-Key Part P332KDACT-ND -> P30.1KDACT-ND
- R29, R31, R34, R36: Digi-Key Part (none) -> P10KDACT-ND
- U10, U12, U19: Digi-Key Part 296-47385-1-ND -> 296-1282-1-ND
- U11: Digi-Key Part (none) -> 296-25227-1-ND
Changed lines of the file:
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@@
       (effects (font (size 1.27 1.27)) hide)
     )
-    (property "Digi-Key Part" "296-47385-1-ND" (id 4) (at 213.36 137.16 0)
+    (property "Digi-Key Part" "296-1282-1-ND" (id 4) (at 213.36 137.16 0)
       (effects (font (size 1.27 1.27)) hide)
     )
@@
       (effects (font (size 1.27 1.27)) hide)
     )
-    (property "Digi-Key Part" "296-47385-1-ND" (id 4) (at 227.33 137.16 0)
+    (property "Digi-Key Part" "296-1282-1-ND" (id 4) (at 227.33 137.16 0)
       (effects (font (size 1.27 1.27)) hide)
     )
@@
     )
     (property "LCSC Part #" "C193969" (id 4) (at 205.105 80.645 0)
+      (effects (font (size 1.27 1.27)) hide)
+    )
+    (property "Digi-Key Part" "296-25227-1-ND" (id 5) (at 205.105 80.645 0)
       (effects (font (size 1.27 1.27)) hide)
     )
@@
       (effects (font (size 1.27 1.27)) hide)
     )
-    (property "Digi-Key Part" "296-47385-1-ND" (id 4) (at 116.205 48.26 0)
+    (property "Digi-Key Part" "296-1282-1-ND" (id 4) (at 116.205 48.26 0)
       (effects (font (size 1.27 1.27)) hide)
     )
@@
       (effects (font (size 1.27 1.27)) hide)
     )
-    (property "Digi-Key Part" "" (id 4) (at 100.965 114.935 90)
+    (property "Digi-Key Part" "P10KDACT-ND" (id 4) (at 100.965 114.935 90)
       (effects (font (size 1.27 1.27)) hide)
     )
@@
       (effects (font (size 1.27 1.27)) hide)
     )
-    (property "Digi-Key Part" "296-47385-1-ND" (id 4) (at 116.205 117.475 0)
+    (property "Digi-Key Part" "296-1282-1-ND" (id 4) (at 116.205 117.475 0)
       (effects (font (size 1.27 1.27)) hide)
     )
@@
       (effects (font (size 1.27 1.27)) hide)
     )
-    (property "Digi-Key Part" "" (id 4) (at 118.11 107.315 90)
+    (property "Digi-Key Part" "P10KDACT-ND" (id 4) (at 118.11 107.315 90)
       (effects (font (size 1.27 1.27)) hide)
     )
@@
       (effects (font (size 1.27 1.27)) hide)
     )
-    (property "Digi-Key Part" "P332KDACT-ND" (id 4) (at 100.965 107.315 90)
+    (property "Digi-Key Part" "P30.1KDACT-ND" (id 4) (at 100.965 107.315 90)
       (effects (font (size 1.27 1.27)) hide)
     )
@@
       (effects (font (size 1.27 1.27)) hide)
     )
-    (property "Digi-Key Part" "P332KDACT-ND" (id 4) (at 100.965 38.1 90)
+    (property "Digi-Key Part" "P30.1KDACT-ND" (id 4) (at 100.965 38.1 90)
       (effects (font (size 1.27 1.27)) hide)
     )
@@
       (effects (font (size 1.27 1.27)) hide)
     )
-    (property "Digi-Key Part" "296-47385-1-ND" (id 4) (at 116.205 150.495 0)
+    (property "Digi-Key Part" "296-1282-1-ND" (id 4) (at 116.205 150.495 0)
       (effects (font (size 1.27 1.27)) hide)
     )
@@
       (effects (font (size 1.27 1.27)) hide)
     )
-    (property "Digi-Key Part" "296-47385-1-ND" (id 4) (at 165.1 45.72 0)
+    (property "Digi-Key Part" "296-1282-1-ND" (id 4) (at 165.1 45.72 0)
       (effects (font (size 1.27 1.27)) hide)
     )
@@
       (effects (font (size 1.27 1.27)) hide)
     )
-    (property "Digi-Key Part" "" (id 4) (at 117.475 38.1 90)
+    (property "Digi-Key Part" "P10KDACT-ND" (id 4) (at 117.475 38.1 90)
       (effects (font (size 1.27 1.27)) hide)
     )
@@
       (effects (font (size 1.27 1.27)) hide)
     )
-    (property "Digi-Key Part" "" (id 4) (at 100.965 45.72 90)
+    (property "Digi-Key Part" "P10KDACT-ND" (id 4) (at 100.965 45.72 90)
       (effects (font (size 1.27 1.27)) hide)
     )
@@
       (effects (font (size 1.27 1.27)) hide)
     )
-    (property "Digi-Key Part" "296-47385-1-ND" (id 4) (at 116.84 81.28 0)
+    (property "Digi-Key Part" "296-1282-1-ND" (id 4) (at 116.84 81.28 0)
       (effects (font (size 1.27 1.27)) hide)
     )
@@
       (effects (font (size 1.27 1.27)) hide)
     )
-    (property "Digi-Key Part" "296-47385-1-ND" (id 4) (at 165.1 114.935 0)
+    (property "Digi-Key Part" "296-1282-1-ND" (id 4) (at 165.1 114.935 0)
       (effects (font (size 1.27 1.27)) hide)
     )
@@
       (effects (font (size 1.27 1.27)) hide)
     )
-    (property "Digi-Key Part" "296-47385-1-ND" (id 4) (at 219.71 137.16 0)
-      (effects (font (size 1.27 1.27)) hide)
-    )
+    (property "Digi-Key Part" "296-1282-1-ND" (id 4) (at 219.71 137.16 0)
+      (effects (font (size 1.27 1.27)) hide)
+    )
