File: main_board/output_monitors.kicad_sch (KiCad schematic)
At the start: 52 parts, among them U14 TL072CDR, U17 TL072CDR, U18 TL072CDR, U4 TL072CDR

Commit message: Updates bom for digi-key
Parts:
- U14, U17, U18, U4: Digi-Key Part 296-47385-1-ND -> 296-1282-1-ND
Changed lines of the file:
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@@
       (effects (font (size 1.27 1.27)) hide)
     )
-    (property "Digi-Key Part" "296-47385-1-ND" (id 4) (at 57.15 172.72 0)
+    (property "Digi-Key Part" "296-1282-1-ND" (id 4) (at 57.15 172.72 0)
       (effects (font (size 1.27 1.27)) hide)
     )
@@
       (effects (font (size 1.27 1.27)) hide)
     )
-    (property "Digi-Key Part" "296-47385-1-ND" (id 4) (at 180.975 136.525 0)
+    (property "Digi-Key Part" "296-1282-1-ND" (id 4) (at 180.975 136.525 0)
       (effects (font (size 1.27 1.27)) hide)
     )
@@
       (effects (font (size 1.27 1.27)) hide)
     )
-    (property "Digi-Key Part" "296-47385-1-ND" (id 4) (at 180.975 34.925 0)
+    (property "Digi-Key Part" "296-1282-1-ND" (id 4) (at 180.975 34.925 0)
       (effects (font (size 1.27 1.27)) hide)
     )
@@
       (effects (font (size 1.27 1.27)) hide)
     )
-    (property "Digi-Key Part" "296-47385-1-ND" (id 4) (at 36.83 172.72 0)
+    (property "Digi-Key Part" "296-1282-1-ND" (id 4) (at 36.83 172.72 0)
       (effects (font (size 1.27 1.27)) hide)
     )
@@
       (effects (font (size 1.27 1.27)) hide)
     )
-    (property "Digi-Key Part" "296-47385-1-ND" (id 4) (at 95.885 63.5 0)
+    (property "Digi-Key Part" "296-1282-1-ND" (id 4) (at 95.885 63.5 0)
       (effects (font (size 1.27 1.27)) hide)
     )
@@
       (effects (font (size 1.27 1.27)) hide)
     )
-    (property "Digi-Key Part" "296-47385-1-ND" (id 4) (at 180.975 99.695 0)
+    (property "Digi-Key Part" "296-1282-1-ND" (id 4) (at 180.975 99.695 0)
       (effects (font (size 1.27 1.27)) hide)
     )
@@
       (effects (font (size 1.27 1.27)) hide)
     )
-    (property "Digi-Key Part" "296-47385-1-ND" (id 4) (at 95.885 99.06 0)
+    (property "Digi-Key Part" "296-1282-1-ND" (id 4) (at 95.885 99.06 0)
       (effects (font (size 1.27 1.27)) hide)
     )
@@
       (effects (font (size 1.27 1.27)) hide)
     )
-    (property "Digi-Key Part" "296-47385-1-ND" (id 4) (at 46.99 172.72 0)
+    (property "Digi-Key Part" "296-1282-1-ND" (id 4) (at 46.99 172.72 0)
       (effects (font (size 1.27 1.27)) hide)
     )
@@
       (effects (font (size 1.27 1.27)) hide)
     )
-    (property "Digi-Key Part" "296-47385-1-ND" (id 4) (at 95.25 34.925 0)
+    (property "Digi-Key Part" "296-1282-1-ND" (id 4) (at 95.25 34.925 0)
       (effects (font (size 1.27 1.27)) hide)
     )
@@
       (effects (font (size 1.27 1.27)) hide)
     )
-    (property "Digi-Key Part" "296-47385-1-ND" (id 4) (at 180.975 64.135 0)
+    (property "Digi-Key Part" "296-1282-1-ND" (id 4) (at 180.975 64.135 0)
       (effects (font (size 1.27 1.27)) hide)
     )
@@
       (effects (font (size 1.27 1.27)) hide)
     )
-    (property "Digi-Key Part" "296-47385-1-ND" (id 4) (at 67.31 172.72 0)
+    (property "Digi-Key Part" "296-1282-1-ND" (id 4) (at 67.31 172.72 0)
       (effects (font (size 1.27 1.27)) hide)
     )
@@
       (effects (font (size 1.27 1.27)) hide)
     )
-    (property "Digi-Key Part" "296-47385-1-ND" (id 4) (at 95.885 135.89 0)
-      (effects (font (size 1.27 1.27)) hide)
-    )
+    (property "Digi-Key Part" "296-1282-1-ND" (id 4) (at 95.885 135.89 0)
+      (effects (font (size 1.27 1.27)) hide)
+    )
