File: panel/panel.kicad_sch (KiCad schematic)
At the start: 48 parts

Commit message: Ver 2.0 of board.
Also major advances in code.
Parts:
- added H46, H47, H48, H49, H50, H51, H52, H53, H54, H55, H56, H57, H58, H59, H60, H61, H62, H63: MountingHole, panel:3mmLED, symbol Mechanical:MountingHole
Other:
- note added: "Blue Monitor LEDs"
- note added: "Input monitor LEDs"
- note added: "Out0"
- note added: "Out1"
- note added: "Out2"
- note added: "Out3"
- note added: "Out4"
- note added: "Out5"
- note added: "Out6"
- note added: "Out7"
- note added: "Red Monitor LEDs"
- note removed: "Clip LEDs"
- moved on the sheet: H17, H18, H19, H20

Commit message: Updates panel
Other:
- title: (none) -> Bonkulator Panel
Changed lines of the file:
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@@
 (kicad_sch (version 20211123) (generator eeschema)
   (paper "A4")
+  (title_block
+    (title "Bonkulator Panel")
+    (rev "2.1")
+  )
   (junction (at 58.42 64.135) (diameter 0) (color 0 0 0 0)
   )

Commit message: Removes KiCAD logo, moves display outline
Parts:
- GR3: footprint Symbol:KiCad-Logo_5mm_SilkScreen -> panel:bamboo_bonk2
Changed lines of the file:
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@@
   )
   (symbol (lib_id "Graphic:Logo_Open_Hardware_Small") (at 231.775 83.185 0) (unit 1)
-    (in_bom yes) (on_board yes)
+    (in_bom yes) (on_board no)
     (property "Reference" "GR2" (id 0) (at 231.775 76.2 0))
     (property "Value" "Logo_Open_Hardware_Small" (id 1) (at 231.775 88.9 0)
@@
   )
   (symbol (lib_id "greenface-symbols:small_logo") (at 231.14 70.485 0) (unit 1)
-    (in_bom yes) (on_board yes) (fields_autoplaced)
+    (in_bom yes) (on_board no) (fields_autoplaced)
     (property "Reference" "GR3" (id 0) (at 231.14 65.3755 0))
     (property "Value" "small_logo" (id 1) (at 231.14 68.1506 0))
-    (property "Footprint" "Symbol:KiCad-Logo_5mm_SilkScreen" (id 2) (at 231.14 70.485 0)
+    (property "Footprint" "panel:bamboo_bonk2" (id 2) (at 231.14 70.485 0)
       (effects (font (size 1.27 1.27)) hide)
     )
@@
     )
     (path "/e52387aa-9a3c-4f08-b265-477019aca115"
-      (reference "GR3") (unit 1) (value "small_logo") (footprint "Symbol:KiCad-Logo_5mm_SilkScreen")
+      (reference "GR3") (unit 1) (value "small_logo") (footprint "panel:bamboo_bonk2")
     )
     (path "/495b9f3e-72d4-4443-8d1b-2b95612acb36"

Commit message: New front panel silkscreen
Parts:
- GR3: footprint panel:bamboo_bonk2 -> panel:wifi
Changed lines of the file:
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@@
   )
   (symbol (lib_id "Graphic:Logo_Open_Hardware_Small") (at 231.775 83.185 0) (unit 1)
-    (in_bom yes) (on_board no)
+    (in_bom yes) (on_board yes)
     (property "Reference" "GR2" (id 0) (at 231.775 76.2 0))
     (property "Value" "Logo_Open_Hardware_Small" (id 1) (at 231.775 88.9 0)
@@
   )
   (symbol (lib_id "greenface-symbols:small_logo") (at 231.14 70.485 0) (unit 1)
-    (in_bom yes) (on_board no) (fields_autoplaced)
+    (in_bom yes) (on_board yes) (fields_autoplaced)
     (property "Reference" "GR3" (id 0) (at 231.14 65.3755 0))
     (property "Value" "small_logo" (id 1) (at 231.14 68.1506 0))
-    (property "Footprint" "panel:bamboo_bonk2" (id 2) (at 231.14 70.485 0)
+    (property "Footprint" "panel:wifi" (id 2) (at 231.14 70.485 0)
       (effects (font (size 1.27 1.27)) hide)
     )
@@
     )
     (path "/e52387aa-9a3c-4f08-b265-477019aca115"
-      (reference "GR3") (unit 1) (value "small_logo") (footprint "panel:bamboo_bonk2")
+      (reference "GR3") (unit 1) (value "small_logo") (footprint "panel:wifi")
     )
     (path "/495b9f3e-72d4-4443-8d1b-2b95612acb36"
