File: BonkDaddy/BonkDaddy2HP_Board/BonkDaddy2HP_Board.kicad_pcb (KiCad board)
At the start: 2 copper layers, 10 x 110 mm, 25 parts, among them J1 EXP, J2 USB_B_Micro, J3 USB_A, Q3 2N7002, Q4 MMBT5401, SW1 Reset, U1 74AHC14

Commit message: Updated LED resistors
Parts:
- Q4: value MMBT5401 -> MMBT3906
- R1: value 100 -> 620
- R2: value 75 -> 620
- R4: value 68 -> 620
- R5: value 47 -> 620
- R8: value 43K -> 30K
Other:
- board text added: "1.1."
- board text added: "v1.1"
- board text removed: "1.0."
- board text removed: "v1.0"
