File: BonkDaddy/BonkDaddy2HP_Board/BonkDaddy2HP_Board.kicad_sch (KiCad schematic)
At the start: 45 parts, among them J1 EXP, J2 USB_B_Micro, J3 USB_A, Q3 2N7000, Q4 2N3906, SW1 Reset, U1 74AHC04

Commit message: Adds 2HP BonkDaddy. Fixes boms/cpl. Updates Readme
Parts:
- removed C2, C3: 10uF, Capacitor_THT:CP_Radial_D5.0mm_P2.00mm, symbol Device:C_Polarized_Small_US
- removed H3, H4: MountingHole, MountingHole:MountingHole_2.5mm, symbol Mechanical:MountingHole
- removed N3, N4: Nut, MountingHole:MountingHole_2.5mm, symbol Mechanical:MountingHole
- removed Q3: 2N7000, Package_TO_SOT_THT:TO-92_Inline_Wide, symbol Transistor_FET:2N7000
- removed Q4: 2N3906, Package_TO_SOT_THT:TO-92_Inline_Wide, symbol Transistor_BJT:2N3906
- removed SC3, SC4: Screw, MountingHole:MountingHole_2.5mm, symbol Mechanical:MountingHole
- removed SK1: A_14-LC-TT, symbol dk_Sockets-for-ICs-Transistors:A_14-LC-TT
- removed SO3, SO4: Stand-off, MountingHole:MountingHole_2.5mm, symbol Mechanical:MountingHole
- removed W3, W4: Washer, MountingHole:MountingHole_2.5mm, symbol Mechanical:MountingHole
- added C3: 1uF, Capacitor_SMD:C_0805_2012Metric, symbol Device:C_Small
- added Q3: 2N7002, Package_TO_SOT_SMD:SOT-23, symbol Transistor_FET:2N7002
- added Q4: MMBT5401, Package_TO_SOT_SMD:SOT-23, symbol Transistor_BJT:MMBT3906
- C1: value .1uF -> 1uF; footprint Capacitor_THT:C_Rect_L7.0mm_W2.0mm_P5.00mm -> Capacitor_SMD:C_0805_2012Metric;   LCSC Part # (none) -> C28323; Digi-Key Part 399-9877-2-ND -> (none)
- J1: footprint Connector_PinHeader_2.54mm:PinHeader_2x05_P2.54mm_Vertical -> Connector_PinHeader_2.54mm:PinHeader_2x05_P2.54mm_Vertical_SMD;   LCSC Part # (none) -> C124391
- R1: footprint Resistor_THT:R_Axial_DIN0207_L6.3mm_D2.5mm_P10.16mm_Horizontal -> Resistor_SMD:R_0805_2012Metric_Pad1.20x1.40mm_HandSolder;   LCSC Part # (none) -> C17408; Digi-Key Part CF14JT100RCT-ND -> (none)
- R2: footprint Resistor_THT:R_Axial_DIN0207_L6.3mm_D2.5mm_P10.16mm_Horizontal -> Resistor_SMD:R_0805_2012Metric_Pad1.20x1.40mm_HandSolder;   LCSC Part # (none) -> C17820; Digi-Key Part CF14JT75R0CT-ND -> (none)
- R3: footprint Resistor_THT:R_Axial_DIN0207_L6.3mm_D2.5mm_P2.54mm_Vertical -> Resistor_SMD:R_0805_2012Metric_Pad1.20x1.40mm_HandSolder;   LCSC Part # (none) -> C17513; Digi-Key Part 738-CFF14JT1K00CT-ND -> (none)
- R4: footprint Resistor_THT:R_Axial_DIN0207_L6.3mm_D2.5mm_P10.16mm_Horizontal -> Resistor_SMD:R_0805_2012Metric_Pad1.20x1.40mm_HandSolder;   LCSC Part # (none) -> C17802; Digi-Key Part CF14JT68R0CT-ND -> (none)
- R5: footprint Resistor_THT:R_Axial_DIN0207_L6.3mm_D2.5mm_P10.16mm_Horizontal -> Resistor_SMD:R_0805_2012Metric_Pad1.20x1.40mm_HandSolder;   LCSC Part # (none) -> C17714; Digi-Key Part CF14JT47R0CT-ND -> (none)
- R6, R9: footprint Resistor_THT:R_Axial_DIN0207_L6.3mm_D2.5mm_P10.16mm_Horizontal -> Resistor_SMD:R_0805_2012Metric_Pad1.20x1.40mm_HandSolder;   LCSC Part # (none) -> C17414; Digi-Key Part CF14JT10K0CT-ND -> (none)
- R7: value 43K -> 30K; footprint Resistor_THT:R_Axial_DIN0207_L6.3mm_D2.5mm_P10.16mm_Horizontal -> Resistor_SMD:R_0805_2012Metric_Pad1.20x1.40mm_HandSolder;   LCSC Part # (none) -> C17621; Digi-Key Part CF14JT43K0CT-ND -> (none)
- R8: footprint Resistor_THT:R_Axial_DIN0207_L6.3mm_D2.5mm_P10.16mm_Horizontal -> Resistor_SMD:R_0805_2012Metric_Pad1.20x1.40mm_HandSolder;   LCSC Part # (none) -> C17695; Digi-Key Part CF14JT43K0CT-ND -> (none)
- U1: value 74AHC04 -> 74AHC14; footprint Package_DIP:DIP-14_W7.62mm_Socket -> Package_SO:SOIC-14_3.9x8.7mm_P1.27mm;   LCSC Part # (none) -> C5605; Digi-Key Part 296-12772-5-ND -> (none)
Connections:
- net +12V: now also C3.1
- net +3V3: now also U1.13
- net GND: now also R6.2, C3.2, Q3.2 (S); no longer R6.1, U1.13
- net at D2.2 (A), J3.1 (VBUS): now also Q4.3 (C)
- net at J2.1 (VBUS), R8.2: now also Q4.2 (E)
- net at R8.1, R9.2: now also Q4.1 (B)
- net at R7.1: now also R6.1, Q3.1 (G); no longer R6.2
- net at R9.1: now also Q3.3 (D)
Other:
- moved on the sheet: U1E, U1F

Commit message: Adds USB connector to Bonk Daddy 2HP LCSC bom
Parts:
- J3:   LCSC Part # (none) -> C718031
Changed lines of the file:
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@@
+      (effects (font (size 1.27 1.27)) hide)
+    )
+    (property "  LCSC Part #" "C718031" (id 5) (at 209.55 75.565 0)
       (effects (font (size 1.27 1.27)) hide)
     )

Commit message: Uses generate_boms.bat now.
Parts:
- C1, C3:   LCSC Part # C28323 -> (none); LCSC Part # (none) -> C28323
- J1:   LCSC Part # C124391 -> (none); LCSC Part # (none) -> C124391
- J3:   LCSC Part # C718031 -> (none); LCSC Part # (none) -> C718031
- Q3:   LCSC Part # C8545 -> (none); LCSC Part # (none) -> C8545
- Q4:   LCSC Part # C8326 -> (none); LCSC Part # (none) -> C8326
- R1:   LCSC Part # C17408 -> (none); LCSC Part # (none) -> C17408
- R2:   LCSC Part # C17820 -> (none); LCSC Part # (none) -> C17820
- R3:   LCSC Part # C17513 -> (none); LCSC Part # (none) -> C17513
- R4:   LCSC Part # C17802 -> (none); LCSC Part # (none) -> C17802
- R5:   LCSC Part # C17714 -> (none); LCSC Part # (none) -> C17714
- R6, R9:   LCSC Part # C17414 -> (none); LCSC Part # (none) -> C17414
- R7:   LCSC Part # C17621 -> (none); LCSC Part # (none) -> C17621
- R8:   LCSC Part # C17695 -> (none); LCSC Part # (none) -> C17695
- U1:   LCSC Part # C5605 -> (none); LCSC Part # (none) -> C5605
Changed lines of the file:
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@@
       (effects (font (size 1.27 1.27)) hide)
     )
-    (property "  LCSC Part #" "C17802" (id 5) (at 124.46 88.9 0)
+    (property "LCSC Part #" "C17802" (id 5) (at 124.46 88.9 0)
       (effects (font (size 1.27 1.27)) hide)
     )
@@
       (effects (font (size 1.27 1.27)) hide)
     )
-    (property "  LCSC Part #" "C17408" (id 5) (at 41.275 84.455 0)
+    (property "LCSC Part #" "C17408" (id 5) (at 41.275 84.455 0)
       (effects (font (size 1.27 1.27)) hide)
     )
@@
       (effects (font (size 1.27 1.27)) hide)
     )
-    (property "  LCSC Part #" "C718031" (id 5) (at 209.55 75.565 0)
+    (property "LCSC Part #" "C718031" (id 5) (at 209.55 75.565 0)
       (effects (font (size 1.27 1.27)) hide)
     )
@@
       (effects (font (size 1.27 1.27)) hide)
     )
-    (property "  LCSC Part #" "C17414" (id 5) (at 244.475 73.66 0)
+    (property "LCSC Part #" "C17414" (id 5) (at 244.475 73.66 0)
       (effects (font (size 1.27 1.27)) hide)
     )
@@
       (effects (font (size 1.27 1.27)) hide)
     )
-    (property "  LCSC Part #" "C5605" (id 5) (at 81.915 152.4 0)
+    (property "LCSC Part #" "C5605" (id 5) (at 81.915 152.4 0)
       (effects (font (size 1.27 1.27)) hide)
     )
@@
       (effects (font (size 1.27 1.27)) hide)
     )
-    (property "  LCSC Part #" "C17513" (id 5) (at 196.85 107.315 0)
+    (property "LCSC Part #" "C17513" (id 5) (at 196.85 107.315 0)
       (effects (font (size 1.27 1.27)) hide)
     )
@@
       (effects (font (size 1.27 1.27)) hide)
     )
-    (property "  LCSC Part #" "C5605" (id 5) (at 51.435 152.4 0)
+    (property "LCSC Part #" "C5605" (id 5) (at 51.435 152.4 0)
       (effects (font (size 1.27 1.27)) hide)
     )
@@
       (effects (font (size 1.27 1.27)) hide)
     )
-    (property "  LCSC Part #" "C28323" (id 5) (at 259.715 73.025 0)
+    (property "LCSC Part #" "C28323" (id 5) (at 259.715 73.025 0)
       (effects (font (size 1.27 1.27)) hide)
     )
@@
       (effects (font (size 1.27 1.27)) hide)
     )
-    (property "  LCSC Part #" "C8326" (id 5) (at 183.515 67.945 0)
+    (property "LCSC Part #" "C8326" (id 5) (at 183.515 67.945 0)
       (effects (font (size 1.27 1.27)) hide)
     )
@@
       (effects (font (size 1.27 1.27)) hide)
     )
-    (property "  LCSC Part #" "C28323" (id 5) (at 105.41 156.845 0)
+    (property "LCSC Part #" "C28323" (id 5) (at 105.41 156.845 0)
       (effects (font (size 1.27 1.27)) hide)
     )
@@
       (effects (font (size 1.27 1.27)) hide)
     )
-    (property "  LCSC Part #" "C17820" (id 5) (at 114.935 62.23 0)
+    (property "LCSC Part #" "C17820" (id 5) (at 114.935 62.23 0)
       (effects (font (size 1.27 1.27)) hide)
     )
@@
       (effects (font (size 1.27 1.27)) hide)
     )
-    (property "  LCSC Part #" "C124391" (id 5) (at 81.915 88.9 0)
+    (property "LCSC Part #" "C124391" (id 5) (at 81.915 88.9 0)
       (effects (font (size 1.27 1.27)) hide)
     )
@@
       (effects (font (size 1.27 1.27)) hide)
     )
-    (property "  LCSC Part #" "C5605" (id 5) (at 59.055 91.44 0)
+    (property "LCSC Part #" "C5605" (id 5) (at 59.055 91.44 0)
       (effects (font (size 1.27 1.27)) hide)
     )
@@
       (effects (font (size 1.27 1.27)) hide)
     )
-    (property "  LCSC Part #" "C8545" (id 5) (at 235.585 61.595 0)
+    (property "LCSC Part #" "C8545" (id 5) (at 235.585 61.595 0)
       (effects (font (size 1.27 1.27)) hide)
     )
@@
       (effects (font (size 1.27 1.27)) hide)
     )
-    (property "  LCSC Part #" "C5605" (id 5) (at 121.92 152.4 0)
+    (property "LCSC Part #" "C5605" (id 5) (at 121.92 152.4 0)
       (effects (font (size 1.27 1.27)) hide)
     )
@@
       (effects (font (size 1.27 1.27)) hide)
     )
-    (property "  LCSC Part #" "C17414" (id 5) (at 194.31 50.165 0)
+    (property "LCSC Part #" "C17414" (id 5) (at 194.31 50.165 0)
       (effects (font (size 1.27 1.27)) hide)
     )
@@
       (effects (font (size 1.27 1.27)) hide)
     )
-    (property "  LCSC Part #" "C5605" (id 5) (at 103.505 73.66 0)
+    (property "LCSC Part #" "C5605" (id 5) (at 103.505 73.66 0)
       (effects (font (size 1.27 1.27)) hide)
     )
@@
       (effects (font (size 1.27 1.27)) hide)
     )
-    (property "  LCSC Part #" "C17621" (id 5) (at 250.825 61.595 90)
+    (property "LCSC Part #" "C17621" (id 5) (at 250.825 61.595 90)
       (effects (font (size 1.27 1.27)) hide)
     )
@@
       (effects (font (size 1.27 1.27)) hide)
     )
-    (property "  LCSC Part #" "C17714" (id 5) (at 53.34 64.135 0)
+    (property "LCSC Part #" "C17714" (id 5) (at 53.34 64.135 0)
       (effects (font (size 1.27 1.27)) hide)
     )
@@
       (effects (font (size 1.27 1.27)) hide)
     )
-    (property "  LCSC Part #" "C5605" (id 5) (at 103.505 93.98 0)
+    (property "LCSC Part #" "C5605" (id 5) (at 103.505 93.98 0)
       (effects (font (size 1.27 1.27)) hide)
     )
@@
       (effects (font (size 1.27 1.27)) hide)
     )
-    (property "  LCSC Part #" "C17695" (id 5) (at 175.26 59.69 0)
+    (property "LCSC Part #" "C17695" (id 5) (at 175.26 59.69 0)
       (effects (font (size 1.27 1.27)) hide)
     )
@@
       (effects (font (size 1.27 1.27)) hide)
     )
-    (property "  LCSC Part #" "C5605" (id 5) (at 64.135 73.66 0)
-      (effects (font (size 1.27 1.27)) hide)
-    )
+    (property "LCSC Part #" "C5605" (id 5) (at 64.135 73.66 0)
+      (effects (font (size 1.27 1.27)) hide)
+    )

Commit message: Updated LED resistors
Parts:
- C1, C3: Digi-Key Part (none) -> 1276-1066-1-ND
- J3: LCSC Part # C718031 -> C386737
- Q3: Digi-Key Part (none) -> 4878-2N7002CT-ND
- Q4: value MMBT5401 -> MMBT3906; Digi-Key Part (none) -> MMBT3906LT1GOSCT-ND; LCSC Part # C8326 -> C266589
- R1: value 100 -> 620; Digi-Key Part (none) -> RMCF0805FT620RCT-ND; LCSC Part # C17408 -> C17782
- R2: value 75 -> 620; Digi-Key Part (none) -> RMCF0805FT620RCT-ND; LCSC Part # C17820 -> C17782
- R3: Digi-Key Part (none) -> 311-1.00KCRCT-ND
- R4: value 68 -> 620; Digi-Key Part (none) -> RMCF0805FT620RCT-ND; LCSC Part # C17802 -> C17782
- R5: value 47 -> 620; Digi-Key Part (none) -> RMCF0805FT620RCT-ND; LCSC Part # C17714 -> C17782
- R6, R9: Digi-Key Part (none) -> RMCF0805FT10K0CT-ND
- R7: Digi-Key Part (none) -> RMCF0805FT30K0CT-ND
- R8: value 43K -> 30K; Digi-Key Part (none) -> RMCF0805FT30K0CT-ND; LCSC Part # C17695 -> C17621
- U1: Digi-Key Part (none) -> 296-9179-1-ND
Other:
- note added: "Amphenol UE27AE54100"
